File: hardware/bolt_logic/wifi.kicad_sch (KiCad schematic)
At the start: 7 parts, among them J4 ESP PROG, U30 ESP32-WROOM-32

Commit message: Schematic: ESP32-WROOM-32UE (u.FL) instead of WROOM-32
The board sits inside the aluminium inverter housing, where an on-module
PCB antenna would not radiate, and the WROOM-32 antenna keep-out did not
fit the layout. The UE variant is pin-identical with a u.FL connector for
an external antenna. Netlist re-verified against the design table.

Co-Authored-By: Claude Opus 5.5 <noreply@anthropic.com>
Claude-Session: https://claude.ai/code/session_01KW1M8KfVLc83FDDiK2YEWM
Parts:
- U30: value ESP32-WROOM-32 -> ESP32-WROOM-32UE; footprint RF_Module:ESP32-WROOM-32 -> RF_Module:ESP32-WROOM-32UE; symbol RF_Module:ESP32-WROOM-32 -> RF_Module:ESP32-WROOM-32UE
Connections:
- no-connect marks 29 -> 23
Changed lines of the file:
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@@
     (at 58.42 63.5)
-)
-  (no_connect
-    (at 27.94 81.28)
-)
-  (no_connect
-    (at 27.94 83.82)
-)
-  (no_connect
-    (at 27.94 88.9)
 )
   (wire
@@
         (font (size 1.27 1.27)) hide)))
   (no_connect
-    (at 27.94 86.36)
-)
-  (no_connect
-    (at 27.94 76.2)
-)
-  (no_connect
-    (at 27.94 78.74)
-)
-  (no_connect
     (at 58.42 68.58)
 )
@@
         (font (size 1.27 1.27)) hide)))
   (symbol
-    (lib_id "RF_Module:ESP32-WROOM-32")
+    (lib_id "RF_Module:ESP32-WROOM-32UE")
     (at 43.18 76.2 0)
     (unit 1)
@@
         (font (size 1.27 1.27))
         (justify left)))
-    (property "Value" "ESP32-WROOM-32"
+    (property "Value" "ESP32-WROOM-32UE"
       (at 27.94 114.16 0)
       (effects
         (font (size 1.27 1.27))
         (justify left)))
-    (property "Footprint" "RF_Module:ESP32-WROOM-32"
+    (property "Footprint" "RF_Module:ESP32-WROOM-32UE"
       (at 43.18 76.2 0)
       (effects
