File: hardware/bolt_logic/power.kicad_sch (KiCad schematic)
At the start: 45 parts, among them Q1 BTS443P, Q2 BTS443P, U1 AP63205WU, U2 LD1117S33TR

Commit message: Fix BTS443P input drive with 2N7002 pull-downs (Q3, Q4); re-route
The BTS443P has no GND pin and switches on when IN is pulled to ground (input switch
sinks 0.7-1.2 mA; < 50 uA keeps it off). The schematic drove IN like a logic input:
Q1's IN went to GND through 6.8k (always on, regardless of ignition) and Q2's IN to
PA15 through 1k (gate power could never be switched off).

Owner-approved fix: a 2N7002 from each IN to GND. Q3's gate comes from the existing IGN
divider (10k/6.8k); Q4's from PA15 through R4, with the existing R5 (10k) holding it
off while PA15 is still JTDI with its internal pull-up at reset. Firmware polarity and
board detection are unchanged.

Re-placed and re-routed: 0 unconnected, DRC clean (also at 0.20 mm clearance); the
buck block is unchanged and locked. A reference that lands on its own pin-1 mark is
now slid clear (clear_own_silk). Schematic PDF regenerated.

Co-Authored-By: Claude Opus 5.5 <noreply@anthropic.com>
Claude-Session: https://claude.ai/code/session_01KW1M8KfVLc83FDDiK2YEWM
Parts:
- added Q3, Q4: 2N7002, Package_TO_SOT_SMD:SOT-23, symbol Transistor_FET:2N7002
Connections:
- net GND: now also Q3.2 (S), Q4.2 (S)
- net Q1_IN: now also Q3.3 (D); no longer R1.2, R2.1
- net Q2_IN: now also Q4.3 (D); no longer R4.2
- new net Q1_G: Q3.1 (G), R1.2, R2.1
- new net Q2_G: Q4.1 (G), R4.2
Other:
- moved on the sheet: C1, C10, C11, C12, C13, C14, C15, C16, C2, C3, C4, C5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

Commit message: Use JLCPCB-stocked parts: BTS6143D, 74HCT10, TCA0372 (schematic)
Owner-approved part changes so JLCPCB can assemble the board:
- Q1/Q2 BTS443P -> BTS6143D: same PG-TO252-5-11 pinout and IN-to-GND input, so the
  symbol, footprint and Q3/Q4 drive are unchanged (BOM only).
- U6 CD74HCT30 -> 74HCT10: PWM_INHIBIT = NAND(GATE_OK_5V, GATE_FLT_F, OCUR_OK), the
  same logic since U5 already ANDs HEALTH1-4.
- U13 L272D -> onsemi TCA0372DW (SOIC-16W), new custom symbol; exciter values unchanged.
- BOM: 3.3 nF C0G -> Murata GRM2165C1H332JA01D (previous choice out of stock);
  74HCT4052 -> TI CD74HCT4052M96 C469908 (confirmed listing); BTS133TC kept (owner).

The routed board and regenerated fab files follow once the routing run completes;
until then fab/ on this branch reflects the previous schematic.

Co-Authored-By: Claude Opus 5.5 <noreply@anthropic.com>
Claude-Session: https://claude.ai/code/session_01KW1M8KfVLc83FDDiK2YEWM
Parts:
- Q1, Q2: value BTS443P -> BTS6143D
Changed lines of the file:
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@@
         (font (size 1.27 1.27))
         (justify left)))
-    (property "Value" "BTS443P"
+    (property "Value" "BTS6143D"
       (at 55.88 53.2 0)
       (effects
@@
         (font (size 1.27 1.27))
         (justify left)))
-    (property "Value" "BTS443P"
+    (property "Value" "BTS6143D"
       (at 35.56 93.84 0)
       (effects
