File: hardware/bolt_logic/resolver.kicad_sch (KiCad schematic)
At the start: 55 parts, among them U12 MCP6292, U13 L272D, U14 MCP6292

Commit message: Use JLCPCB-stocked parts: BTS6143D, 74HCT10, TCA0372 (schematic)
Owner-approved part changes so JLCPCB can assemble the board:
- Q1/Q2 BTS443P -> BTS6143D: same PG-TO252-5-11 pinout and IN-to-GND input, so the
  symbol, footprint and Q3/Q4 drive are unchanged (BOM only).
- U6 CD74HCT30 -> 74HCT10: PWM_INHIBIT = NAND(GATE_OK_5V, GATE_FLT_F, OCUR_OK), the
  same logic since U5 already ANDs HEALTH1-4.
- U13 L272D -> onsemi TCA0372DW (SOIC-16W), new custom symbol; exciter values unchanged.
- BOM: 3.3 nF C0G -> Murata GRM2165C1H332JA01D (previous choice out of stock);
  74HCT4052 -> TI CD74HCT4052M96 C469908 (confirmed listing); BTS133TC kept (owner).

The routed board and regenerated fab files follow once the routing run completes;
until then fab/ on this branch reflects the previous schematic.

Co-Authored-By: Claude Opus 5.5 <noreply@anthropic.com>
Claude-Session: https://claude.ai/code/session_01KW1M8KfVLc83FDDiK2YEWM
Parts:
- removed unit 3 of U13
- removed unit 2 of U13
- U13: value L272D -> TCA0372DW; footprint Package_SO:SOIC-16_3.9x9.9mm_P1.27mm -> Package_SO:SOIC-16W_7.5x10.3mm_P1.27mm; symbol Amplifier_Operational:L272D -> Bolt:TCA0372
Connections:
- net EXC_AC: now also U13.9 (+INA); no longer U13.13 (+)
- net EXC_FBA: now also U13.10 (-INA); no longer U13.14 (-)
- net EXC_FBB: now also U13.7 (-INB)
- net EXC_OA: now also U13.16 (OUTA); no longer U13.3
- net EXC_OB: now also U13.2 (OUTB)
- net EXC_VB: now also U13.8 (+INB)
- net GND: now also U13.12 (GND), U13.13 (GND), U13.4 (GND), U13.5 (GND)
- net VCC_12V: now also U13.1 (VCC)
- no-connect marks 0 -> 5
Other:
- moved on the sheet: C78, C79, C80, C81, C82, C83, C84, C85, C86, C87, C88, C89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
