File: hardware/bolt_logic/bolt_logic.kicad_pcb (KiCad board)
At the start: 4 copper layers, 289 x 112 mm, 241 parts, among them CN1 GM X1 48-way, CN2 SSW-120-01-T-D-LL, J1 SWD, J4 ESP PROG, Q1 BTS443P, Q2 BTS443P, U1 AP63205WU, U10 LM2901, U11 74HCT4052, U12 MCP6292, U13 L272D, U14 MCP6292, U2 LD1117S33TR, U20 BTS133TC, U21 BTS133TC, U22 BTS133TC, U23 SN65HVD234, U3 STM32F103RBT6, U30 ESP32-WROOM-32E, U4 74HCT573, U5 74HC21, U6 CD74HCT30, U7 MCP6292, U8 MCP6292, U9 LM2901, Y1 8MHz, Y2 32.768kHz

Commit message: Fix BTS443P input drive with 2N7002 pull-downs (Q3, Q4); re-route
The BTS443P has no GND pin and switches on when IN is pulled to ground (input switch
sinks 0.7-1.2 mA; < 50 uA keeps it off). The schematic drove IN like a logic input:
Q1's IN went to GND through 6.8k (always on, regardless of ignition) and Q2's IN to
PA15 through 1k (gate power could never be switched off).

Owner-approved fix: a 2N7002 from each IN to GND. Q3's gate comes from the existing IGN
divider (10k/6.8k); Q4's from PA15 through R4, with the existing R5 (10k) holding it
off while PA15 is still JTDI with its internal pull-up at reset. Firmware polarity and
board detection are unchanged.

Re-placed and re-routed: 0 unconnected, DRC clean (also at 0.20 mm clearance); the
buck block is unchanged and locked. A reference that lands on its own pin-1 mark is
now slid clear (clear_own_silk). Schematic PDF regenerated.

Co-Authored-By: Claude Opus 5.5 <noreply@anthropic.com>
Claude-Session: https://claude.ai/code/session_01KW1M8KfVLc83FDDiK2YEWM
Parts:
- added Q3: 2N7002, Package_TO_SOT_SMD:SOT-23, F.Cu at (76.7, 107.6)
- added Q4: 2N7002, Package_TO_SOT_SMD:SOT-23, F.Cu at (89.7, 113.0)
- moved C87 47.2 mm to (82.8, 123.3), turned to 90 degrees
- moved C79 46.6 mm to (88.8, 123.3), turned to 90 degrees
- moved C78 46.0 mm to (129.1, 125.3), turned to 0 degrees
- moved C77 35.8 mm to (93.8, 123.1), turned to 180 degrees
- moved R72 30.1 mm to (117.2, 140.5), turned to 180 degrees
- moved C84 26.8 mm to (135.2, 124.0)
- moved R71 25.5 mm to (119.5, 136.0), turned to -90 degrees
- moved R70 21.7 mm to (115.0, 135.3), turned to 180 degrees
- moved C88 14.8 mm to (133.7, 130.7)
- moved R82 11.3 mm to (121.7, 148.0), turned to -90 degrees
- moved R83 9.81 mm to (127.0, 143.5), turned to -90 degrees
- moved C80 9.60 mm to (138.4, 129.4), turned to -90 degrees
- moved R91 9.49 mm to (130.7, 136.0)
- moved C86 9.03 mm to (141.2, 139.0)
- moved R68 8.31 mm to (100.0, 132.3), turned to 180 degrees
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Connections:
- R1 pad 2: Q1_IN -> Q1_G
- R2 pad 1: Q1_IN -> Q1_G
- R4 pad 2: Q2_IN -> Q2_G
Routing:
- net ENC_A_F: track 62.2 -> 17.2 mm, vias 2 -> 0
- net +3V3: track 437.4 -> 477.3 mm, vias 9 -> 8
- net Q2_G: track 0.00 -> 26.4 mm
- net FWD_IN: track 66.6 -> 91.7 mm
- net HEALTH4_F: track 48.6 -> 23.5 mm, vias 0 -> 2
- net CRUISE_IN: track 53.7 -> 78.2 mm
- net EXC_OA: track 18.6 -> 41.1 mm, vias 0 -> 4
- net Q2_IN: track 27.5 -> 5.10 mm, vias 2 -> 0
- net EXC_FBB: track 25.7 -> 47.4 mm, vias 2 -> 3
- net BRAKE_IN: track 84.7 -> 64.4 mm, vias 3 -> 2
- net ENC_5V: track 163.0 -> 143.2 mm
- net NRST: track 47.5 -> 27.8 mm
- net PUMP_OUT_SW: track 215.5 -> 197.0 mm, vias 1 -> 3
- net PRECHARGE_OUT: track 93.4 -> 111.3 mm, vias 2 -> 4
- net IGN: track 149.3 -> 166.7 mm, vias 3 -> 2
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
Commit message: Silkscreen: owner's board text, CN1/CN2 outlines and pin labels
Adds the owner's text block (OPEN INVERTER / CHEVY BOLT INVERTER LOGIC BOARD V0.1 /
OPENINVERTER.ORG / COPYRIGHT 2026 / authors) in the empty area right of the MCU,
reserved from placement (TEXT_AREA). CN1 and CN2 footprints had no silkscreen: CN1 now
has an outline, row letters A-M, pin 1 and its reference; CN2 an outline and pins
1/2/39/40 on both sides (soldered from the top) and its reference on the bottom.
Silk only, no copper change; DRC unchanged; fab files regenerated.

Co-Authored-By: Claude Opus 5.5 <noreply@anthropic.com>
Claude-Session: https://claude.ai/code/session_01KW1M8KfVLc83FDDiK2YEWM
Other:
- board text added: "1"
- board text added: "2"
- board text added: "39"
- board text added: "40"
- board text added: "A"
- board text added: "B"
- board text added: "C"
- board text added: "CHEVY BOLT INVERTER LOGIC BOARD V0.1"
- board text added: "CN2 (fitted on bottom)"
- board text added: "COPYRIGHT 2026"
- board text added: "D"
- board text added: "D. MAGUIRE"
- board text added: "E"
- board text added: "F"
- board text added: "G"
- board text added: "H"
- board text added: "I. KELLY"
- board text added: "J"
- board text added: "J. HUEBNER"
- board text added: "K"
- board text added: "L"
- board text added: "M"
- board text added: "OPEN INVERTER"
- board text added: "OPENINVERTER.ORG"
- board text added: "P.S.MANGELSDORF VIA CLAUDE"
Changed lines of the file:
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@@
   (footprint "Bolt:CN1_GM_48pos_4x12" (layer "F.Cu")
     (at 60.3 126.75)
-    (fp_text reference "CN1" (at 0 0) (layer "F.Fab")
-        (effects (font (size 1.27 1.27) (thickness 0.15)))
+    (fp_text reference "CN1" (at -2.8 -4.05) (layer "F.SilkS")
+        (effects (font (size 1.5 1.5) (thickness 0.2)))
     )
     (fp_text value "GM X1 48-way" (at 0 0) (layer "F.Fab") hide
@@
   (footprint "Bolt:CN2_2x20_P2.54_Receptacle_Back" (layer "B.Cu")
     (at 107.729999 184.18 180)
-    (fp_text reference "CN2" (at 0 0) (layer "B.Fab")
-        (effects (font (size 1.27 1.27) (thickness 0.15)) (justify mirror))
+    (fp_text reference "CN2" (at 24.129999 -5.59) (layer "B.SilkS")
+        (effects (font (size 1.5 1.5) (thickness 0.2)) (justify mirror))
     )
     (fp_text value "SSW-120-01-T-D-LL" (at 0 0) (layer "B.Fab") hide
@@
       (net 66 "GND"))
   )
+  (gr_line (start 109.18 182.73) (end 58.019999 182.73)
+    (stroke (width 0.15) (type default)) (layer "B.SilkS"))
+  (gr_line (start 58.019999 188.17) (end 109.18 188.17)
+    (stroke (width 0.15) (type default)) (layer "B.SilkS"))
+  (gr_line (start 58.019999 182.73) (end 58.019999 188.17)
+    (stroke (width 0.15) (type default)) (layer "B.SilkS"))
+  (gr_line (start 109.18 188.17) (end 109.18 182.73)
+    (stroke (width 0.15) (type default)) (layer "B.SilkS"))
+  (gr_line (start 58.019999 188.17) (end 109.18 188.17)
+    (stroke (width 0.15) (type default)) (layer "F.SilkS"))
+  (gr_line (start 61.75 125.3) (end 46.85 125.3)
+    (stroke (width 0.15) (type default)) (layer "F.SilkS"))
+  (gr_line (start 46.85 125.3) (end 46.85 157.9)
+    (stroke (width 0.15) (type default)) (layer "F.SilkS"))
+  (gr_line (start 58.019999 182.73) (end 58.019999 188.17)
+    (stroke (width 0.15) (type default)) (layer "F.SilkS"))
+  (gr_line (start 109.18 188.17) (end 109.18 182.73)
+    (stroke (width 0.15) (type default)) (layer "F.SilkS"))
+  (gr_line (start 46.85 157.9) (end 61.75 157.9)
+    (stroke (width 0.15) (type default)) (layer "F.SilkS"))
+  (gr_line (start 109.18 182.73) (end 58.019999 182.73)
+    (stroke (width 0.15) (type default)) (layer "F.SilkS"))
+  (gr_line (start 61.75 157.9) (end 61.75 125.3)
+    (stroke (width 0.15) (type default)) (layer "F.SilkS"))
   (gr_line (start 44 167) (end 44 115)
     (stroke (width 0.1) (type default)) (layer "Edge.Cuts"))
@@
   (gr_line (start 55 115) (end 55 93)
     (stroke (width 0.1) (type default)) (layer "Edge.Cuts"))
+  (gr_text "40" (at 56.42 186.72) (layer "B.SilkS")
+    (effects (font (size 1 1) (thickness 0.15)) (justify mirror))
+  )
+  (gr_text "39" (at 56.42 184.18) (layer "B.SilkS")
+    (effects (font (size 1 1) (thickness 0.15)) (justify mirror))
+  )
+  (gr_text "1" (at 110.38 184.18) (layer "B.SilkS")
+    (effects (font (size 1 1) (thickness 0.15)) (justify mirror))
+  )
+  (gr_text "2" (at 110.38 186.72) (layer "B.SilkS")
+    (effects (font (size 1 1) (thickness 0.15)) (justify mirror))
+  )
+  (gr_text "CN2 (fitted on bottom)" (at 83.6 189.57) (layer "F.SilkS")
+    (effects (font (size 1.2 1.2) (thickness 0.15)))
+  )
+  (gr_text "K" (at 62.75 133.9) (layer "F.SilkS")
+    (effects (font (size 1 1) (thickness 0.15)))
+  )
+  (gr_text "H" (at 62.75 138.95) (layer "F.SilkS")
+    (effects (font (size 1 1) (thickness 0.15)))
+  )
+  (gr_text "C" (at 62.75 151.45) (layer "F.SilkS")
+    (effects (font (size 1 1) (thickness 0.15)))
+  )
+  (gr_text "M" (at 62.75 126.75) (layer "F.SilkS")
+    (effects (font (size 1 1) (thickness 0.15)))
+  )
+  (gr_text "P.S.MANGELSDORF VIA CLAUDE" (at 289 168.28) (layer "F.SilkS")
+    (effects (font (size 1.5 1.5) (thickness 0.2)))
+  )
+  (gr_text "39" (at 56.42 184.18) (layer "F.SilkS")
+    (effects (font (size 1 1) (thickness 0.15)))
+  )
+  (gr_text "40" (at 56.42 186.72) (layer "F.SilkS")
+    (effects (font (size 1 1) (thickness 0.15)))
+  )
+  (gr_text "1" (at 110.38 184.18) (layer "F.SilkS")
+    (effects (font (size 1 1) (thickness 0.15)))
+  )
+  (gr_text "L" (at 62.75 130.449999) (layer "F.SilkS")
+    (effects (font (size 1 1) (thickness 0.15)))
+  )
+  (gr_text "D. MAGUIRE" (at 289 161.08) (layer "F.SilkS")
+    (effects (font (size 1.5 1.5) (thickness 0.2)))
+  )
+  (gr_text "J. HUEBNER" (at 289 163.48) (layer "F.SilkS")
+    (effects (font (size 1.5 1.5) (thickness 0.2)))
+  )
+  (gr_text "J" (at 62.75 136.45) (layer "F.SilkS")
+    (effects (font (size 1 1) (thickness 0.15)))
+  )
+  (gr_text "A" (at 62.75 156.45) (layer "F.SilkS")
+    (effects (font (size 1 1) (thickness 0.15)))
+  )
+  (gr_text "F" (at 62.75 143.95) (layer "F.SilkS")
+    (effects (font (size 1 1) (thickness 0.15)))
+  )
+  (gr_text "COPYRIGHT 2026" (at 289 158.68) (layer "F.SilkS")
+    (effects (font (size 1.5 1.5) (thickness 0.2)))
+  )
+  (gr_text "OPEN INVERTER" (at 289 148.12) (layer "F.SilkS")
+    (effects (font (size 3 3) (thickness 0.45)))
+  )
+  (gr_text "G" (at 62.75 141.45) (layer "F.SilkS")
+    (effects (font (size 1 1) (thickness 0.15)))
+  )
+  (gr_text "OPENINVERTER.ORG" (at 289 155.8) (layer "F.SilkS")
+    (effects (font (size 1.8 1.8) (thickness 0.25)))
+  )
+  (gr_text "CHEVY BOLT INVERTER LOGIC BOARD V0.1" (at 289 152.92) (layer "F.SilkS")
+    (effects (font (size 1.8 1.8) (thickness 0.25)))
+  )
+  (gr_text "E" (at 62.75 146.45) (layer "F.SilkS")
+    (effects (font (size 1 1) (thickness 0.15)))
+  )
+  (gr_text "B" (at 62.75 153.95) (layer "F.SilkS")
+    (effects (font (size 1 1) (thickness 0.15)))
+  )
+  (gr_text "1" (at 60.3 124.3) (layer "F.SilkS")
+    (effects (font (size 1 1) (thickness 0.15)))
+  )
+  (gr_text "I. KELLY" (at 289 165.88) (layer "F.SilkS")
+    (effects (font (size 1.5 1.5) (thickness 0.2)))
+  )
+  (gr_text "2" (at 110.38 186.72) (layer "F.SilkS")
+    (effects (font (size 1 1) (thickness 0.15)))
+  )
+  (gr_text "D" (at 62.75 148.95) (layer "F.SilkS")
+    (effects (font (size 1 1) (thickness 0.15)))
+  )
   (segment (start 87.068295 106.889493) (end 87.068295 108.124993) (width 0.75) (layer "F.Cu") (net 1))
   (segment (start 122.349992 100.074994) (end 117.099993 94.824994) (width 0.75) (layer "F.Cu") (net 1))

Commit message: Route the board with the stocked parts; regenerate fab files
Full re-place and re-route with U6 = 74HCT10 and U13 = TCA0372DW (SOIC-16W):
0 unconnected, DRC clean (also at 0.20 mm clearance), buck block intact and locked,
owner's silkscreen text and CN1/CN2 marks in place. fab/ regenerated: JLC BOM 61
lines / 220 placements; only CN1, CN2, J1, J4 are hand-fit (plus U20-U22 if JLCPCB
can't place BTS133TC C2681318). Checked in an independent Gerber reader: all layers
and drill files load and placement points land on the changed parts.

Co-Authored-By: Claude Opus 5.5 <noreply@anthropic.com>
Claude-Session: https://claude.ai/code/session_01KW1M8KfVLc83FDDiK2YEWM
Parts:
- Q1, Q2: value BTS443P -> BTS6143D
- U13: value L272D -> TCA0372DW; footprint Package_SO:SOIC-16_3.9x9.9mm_P1.27mm -> Package_SO:SOIC-16W_7.5x10.3mm_P1.27mm
- U6: value CD74HCT30 -> 74HCT10
- moved R91 45.1 mm to (85.7, 139.0)
- moved C79 45.0 mm to (133.7, 124.0), turned to 0 degrees
- moved C44 25.3 mm to (138.7, 201.2)
- moved R28 24.6 mm to (133.5, 200.5)
- moved R27 24.0 mm to (127.5, 199.8), turned to -90 degrees
- moved R30 23.3 mm to (138.7, 176.5)
- moved R29 23.3 mm to (133.5, 176.5), turned to 0 degrees
- moved C40 21.9 mm to (146.3, 195.3), turned to -90 degrees
- moved C43 20.5 mm to (144.0, 176.5)
- moved R22 19.8 mm to (140.2, 190.8)
- moved C121 18.5 mm to (303.5, 193.7), turned to -90 degrees
- moved R33 18.3 mm to (165.0, 176.5)
- moved C46 16.5 mm to (151.5, 195.3), turned to -90 degrees
- moved TP1 16.4 mm to (148.8, 200.0)
- moved U6 14.9 mm to (156.6, 182.0)
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Connections:
- U13 pad 1: (no net) -> VCC_12V
- U13 pad 10: (no net) -> EXC_FBA
- U13 pad 11: EXC_FBB -> (no net)
- U13 pad 12: EXC_VB -> GND
- U13 pad 13: EXC_AC -> GND
- U13 pad 14: EXC_FBA -> (no net)
- U13 pad 16: (no net) -> EXC_OA
- U13 pad 2: (no net) -> EXC_OB
- U13 pad 3: EXC_OA -> (no net)
- U13 pad 4: VCC_12V -> GND
- U13 pad 5: EXC_OB -> GND
- U13 pad 6: GND -> (no net)
- U13 pad 7: (no net) -> EXC_FBB
- U13 pad 8: (no net) -> EXC_VB
- U13 pad 9: (no net) -> EXC_AC
- U6 pad 1: GATE_FLT_F -> GATE_OK_5V
- U6 pad 10: (no net) -> GND
- U6 pad 11: +5V -> GND
- U6 pad 12: +5V -> PWM_INHIBIT
- U6 pad 13: (no net) -> OCUR_OK
- U6 pad 2: HEALTH1_F -> GATE_FLT_F
- U6 pad 3: HEALTH2_F -> GND
- U6 pad 4: HEALTH3_F -> GND
- U6 pad 5: HEALTH4_F -> GND
- U6 pad 6: OCUR_OK -> (no net)
- U6 pad 8: PWM_INHIBIT -> (no net)
- U6 pad 9: (no net) -> GND
Routing:
- net +3V3: track 477.3 -> 539.2 mm, vias 8 -> 10
- net +5V: track 442.4 -> 483.2 mm
- net POS_B: track 99.7 -> 138.2 mm, vias 2 -> 4
- net GATE_FLT: track 46.7 -> 71.4 mm
- net GND: track 272.3 -> 295.4 mm, vias 500 -> 505
- net PUMP_OUT_SW: track 197.0 -> 218.7 mm, vias 3 -> 1
- net HEALTH2_F: track 44.5 -> 23.3 mm, vias 4 -> 3
- net OCUR_OK: track 106.7 -> 85.8 mm, vias 5 -> 4
- net FWD_IN: track 91.7 -> 70.9 mm
- net GATE_FLT_F: track 54.1 -> 34.5 mm
- net UDC: track 32.5 -> 51.4 mm
- net IGN: track 166.7 -> 150.6 mm, vias 2 -> 3
- net GB_AUX: track 88.4 -> 72.4 mm
- net GATE_FLT_MCU: track 58.6 -> 43.0 mm
- net PRECHARGE_OUT: track 111.3 -> 96.7 mm, vias 4 -> 2
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