File: hardware/bolt_logic/bolt_logic.kicad_pcb (KiCad board)
At the start: 4 copper layers, 289 x 112 mm, 243 parts, among them CN1 GM X1 48-way, CN2 SSW-120-01-T-D-LL, J1 SWD, J4 ESP PROG, Q1 BTS6143D, Q2 BTS6143D, Q3 2N7002, Q4 2N7002, U1 AP63205WU, U10 LM2901, U11 74HCT4052, U12 MCP6292, U13 TCA0372DW, U14 MCP6292, U2 LD1117S33TR, U20 BTS133TC, U21 BTS133TC, U22 BTS133TC, U23 SN65HVD234, U3 STM32F103RBT6, U30 ESP32-WROOM-32E, U4 74HCT573, U5 74HC21, U6 74HCT10, U7 MCP6292, U8 MCP6292, U9 LM2901, Y1 8MHz, Y2 32.768kHz

Commit message: BOM: Littelfuse SMBJ26CA for TVS1, SN74ACT10 for U6 (stock)
JLCPCB is out of stock on the Bourns SMBJ26CA (C3719606) and the 74HCT10D (C547236).
- TVS1: Littelfuse SMBJ26CA C83332, same spec and SMB package.
- U6: TI SN74ACT10DR C2861739, same '10 pinout and SOIC-14; ACT has TTL-level inputs
  (VIH 2.0 V) like HCT, so the 3.3 V OCUR_OK line still reads high at 5 V.
No copper change: the routed board only gets U6's value updated; Gerber and drill
artwork is identical to the merged version apart from the generation dates. Schematic,
schematic PDF, fab BOM and docs regenerated.

Co-Authored-By: Claude Opus 5.5 <noreply@anthropic.com>
Claude-Session: https://claude.ai/code/session_01KW1M8KfVLc83FDDiK2YEWM
Parts:
- U6: value 74HCT10 -> SN74ACT10
Changed lines of the file:
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@@
         (effects (font (size 1 1) (thickness 0.15)))
     )
-    (fp_text value "74HCT10" (at 0 5.28 90) (layer "F.Fab")
+    (fp_text value "SN74ACT10" (at 0 5.28 90) (layer "F.Fab")
         (effects (font (size 1 1) (thickness 0.15)))
     )
